Commit message: complete

File: xacro/barista_2.urdf.xacro (robot description, xacro)
@@ -52,5 +52,5 @@
     <parent link="base_link"/>
     <child link="c1"/>
-    <origin xyz="0.0 -0.1  -0.09" rpy="0 1.57 0" />
+    <origin xyz="0.0 -0.1  -0.1" rpy="0 1.57 0" />
   </joint>
 <link name="c2">
@@ -74,5 +74,5 @@
     <parent link="base_link"/>
     <child link="c2"/>
-    <origin xyz="0.0 0.1  -0.09" rpy="0 1.57 0" />
+    <origin xyz="0.0 0.1  -0.1" rpy="0 1.57 0" />
   </joint>
   <!-- Include and instantiate the wheel.xacro macro for the left wheel -->
